File: etl_module_mockup.kicad_pcb (KiCad board)
At the start: 2 copper layers, 43.1 x 56.5 mm, 60 parts, among them J1 WP7B-S040VA1, J2 WP7B-S040VA1, U1 ETROCv2, U2 ETROCv2, U3 ETROCv2, U4 ETROCv2

Commit message: updates
Parts:
- added J1: WP7B-S050VA1-R8000, SamacSys_Parts:WP7BS050VA1R8000, B.Cu at (145.4, 86.5)
- added J2: WP7B-S050VA1-R8000, SamacSys_Parts:WP7BS050VA1R8000, B.Cu at (145.4, 110.0)
- added REF**: crossed_circle_fiducial, unl_silab:crossed_circle_fiducial, F.Cu at (164.9, 125.0)
- added REF**: HV, unl_silab:HV-Pad, F.Cu at (156.2, 125.0)
- added REF**: crossed_circle_fiducial, unl_silab:crossed_circle_fiducial, F.Cu at (164.9, 71.5)
- added REF**: crossed_circle_fiducial, unl_silab:crossed_circle_fiducial, F.Cu at (125.8, 125.0)
- added REF**: HV, unl_silab:HV-Pad, F.Cu at (156.3, 71.5)
- added REF**: HV, unl_silab:HV-Pad, F.Cu at (134.6, 71.5)
- added REF**: HV, unl_silab:HV-Pad, F.Cu at (134.6, 125.0)
- added REF**: crossed_circle_fiducial, unl_silab:crossed_circle_fiducial, F.Cu at (125.8, 71.5)
- added REF**: MountingHole_2.2mm_M2, MountingHole:MountingHole_2.2mm_M2, F.Cu at (145.4, 125.4)
- added REF**: MountingHole_2.2mm_M2, MountingHole:MountingHole_2.2mm_M2, F.Cu at (145.4, 71.1)
- U1, U2, U3, U4: footprint etl_module_mockup:ETROCv2_64pad -> etl_module_mockup:PCB_ETROC2_test; moved to F.Cu
- moved J1 103.8 mm to (33.0, 66.0)
- moved J2 102.5 mm to (34.3, 88.9)
- moved C1 91.5 mm to (34.4, 51.2)
- moved C10 91.5 mm to (41.7, 51.2)
- moved C12 91.5 mm to (36.8, 51.2)
- moved C13 91.5 mm to (65.5, 51.7)
- moved C17 91.5 mm to (60.6, 51.7)
- moved C21 91.5 mm to (67.9, 49.9)
- moved C22 91.5 mm to (65.5, 49.9)
- moved C24 91.5 mm to (60.6, 49.9)
- moved C26 91.5 mm to (50.9, 109.8)
- moved C3 91.5 mm to (41.7, 52.9)
- moved C40 91.5 mm to (29.1, 108.8)
- moved C6 91.5 mm to (36.8, 52.9)
- moved C7 91.5 mm to (34.4, 52.9)
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Routing:
- net /1V2C: track 0.00 -> 98.7 mm, vias 0 -> 4
- net GND: track 0.00 -> 65.9 mm, vias 0 -> 3
- net /1V2D: track 0.00 -> 60.0 mm, vias 0 -> 2
- net /DIN2_P: track 30.6 -> 0.00 mm, vias 1 -> 0
- net /DIN2_N: track 29.4 -> 0.00 mm, vias 1 -> 0
- net /DOUT1_P: track 27.2 -> 0.00 mm, vias 1 -> 0
- net /DOUT1_N: track 27.2 -> 0.00 mm, vias 1 -> 0
- net /DIN3_P: track 23.5 -> 0.00 mm, vias 1 -> 0
- net Net-(J2-Pad16): track 0.00 -> 23.5 mm, vias 0 -> 1
- net /DIN3_N: track 23.5 -> 0.00 mm, vias 1 -> 0
- net /CLK2_P: track 22.4 -> 0.00 mm, vias 1 -> 0
- net /CLK2_N: track 21.8 -> 0.00 mm, vias 1 -> 0
- net /CLK3_P: track 21.2 -> 0.00 mm, vias 1 -> 0
- net /CLK3_N: track 21.2 -> 0.00 mm, vias 1 -> 0
Other:
- board size 43.1 x 56.5 mm -> 139.8 x 74.7 mm
