File: board_to_board.kicad_sch (KiCad schematic)
At the start: 2 parts

Commit message: wip save
Parts:
- J1, J2: renamed from J?; value (none) -> WP7B-S040VA1; footprint (none) -> etl_module_mockup:WP7B-S040VA1
Changed lines of the file:
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@@
   (symbol (lib_id "power:GND") (at 189.23 120.65 0) (unit 1)
     (in_bom yes) (on_board yes)
-    (property "Reference" "#PWR?" (id 0) (at 189.23 127 0)
+    (property "Reference" "#PWR0104" (id 0) (at 189.23 127 0)
       (effects (font (size 1.27 1.27)) hide)
     )
-    (property "Value" "" (id 1) (at 189.357 125.0442 0))
+    (property "Value" "GND" (id 1) (at 189.357 125.0442 0))
     (property "Footprint" "" (id 2) (at 189.23 120.65 0)
       (effects (font (size 1.27 1.27)) hide)
@@
   (symbol (lib_id "power:GND") (at 171.45 120.65 0) (unit 1)
     (in_bom yes) (on_board yes)
-    (property "Reference" "#PWR?" (id 0) (at 171.45 127 0)
+    (property "Reference" "#PWR0105" (id 0) (at 171.45 127 0)
       (effects (font (size 1.27 1.27)) hide)
     )
-    (property "Value" "" (id 1) (at 171.577 125.0442 0))
+    (property "Value" "GND" (id 1) (at 171.577 125.0442 0))
     (property "Footprint" "" (id 2) (at 171.45 120.65 0)
       (effects (font (size 1.27 1.27)) hide)
@@
   (symbol (lib_id "wp7b-s040va1:WP7B-S040VA1") (at 179.07 92.71 0) (unit 1)
     (in_bom yes) (on_board yes)
-    (property "Reference" "J?" (id 0) (at 180.34 61.7982 0))
-    (property "Value" "" (id 1) (at 180.34 64.1096 0))
-    (property "Footprint" "" (id 2) (at 179.07 92.71 0)
+    (property "Reference" "J2" (id 0) (at 180.34 61.7982 0))
+    (property "Value" "WP7B-S040VA1" (id 1) (at 180.34 64.1096 0))
+    (property "Footprint" "etl_module_mockup:WP7B-S040VA1" (id 2) (at 179.07 92.71 0)
       (effects (font (size 1.27 1.27)) hide)
     )
@@
   (symbol (lib_id "power:GND") (at 99.06 121.92 0) (unit 1)
     (in_bom yes) (on_board yes)
-    (property "Reference" "#PWR?" (id 0) (at 99.06 128.27 0)
+    (property "Reference" "#PWR0106" (id 0) (at 99.06 128.27 0)
       (effects (font (size 1.27 1.27)) hide)
     )
-    (property "Value" "" (id 1) (at 99.187 126.3142 0))
+    (property "Value" "GND" (id 1) (at 99.187 126.3142 0))
     (property "Footprint" "" (id 2) (at 99.06 121.92 0)
       (effects (font (size 1.27 1.27)) hide)
@@
   (symbol (lib_id "power:GND") (at 116.84 121.92 0) (unit 1)
     (in_bom yes) (on_board yes)
-    (property "Reference" "#PWR?" (id 0) (at 116.84 128.27 0)
+    (property "Reference" "#PWR0107" (id 0) (at 116.84 128.27 0)
       (effects (font (size 1.27 1.27)) hide)
     )
-    (property "Value" "" (id 1) (at 116.967 126.3142 0))
+    (property "Value" "GND" (id 1) (at 116.967 126.3142 0))
     (property "Footprint" "" (id 2) (at 116.84 121.92 0)
       (effects (font (size 1.27 1.27)) hide)
@@
   (symbol (lib_id "wp7b-s040va1:WP7B-S040VA1") (at 106.68 93.98 0) (unit 1)
     (in_bom yes) (on_board yes)
-    (property "Reference" "J?" (id 0) (at 107.95 63.0682 0))
-    (property "Value" "" (id 1) (at 107.95 65.3796 0))
-    (property "Footprint" "" (id 2) (at 106.68 93.98 0)
+    (property "Reference" "J1" (id 0) (at 107.95 63.0682 0))
+    (property "Value" "WP7B-S040VA1" (id 1) (at 107.95 65.3796 0))
+    (property "Footprint" "etl_module_mockup:WP7B-S040VA1" (id 2) (at 106.68 93.98 0)
       (effects (font (size 1.27 1.27)) hide)
     )
