File: etl_module_mockup.kicad_sch (KiCad schematic)
At the start: 10 parts

Commit message: wip save
Parts:
- R1: value (none) -> 0R; footprint (none) -> Resistor_SMD:R_0201_0603Metric
- R2, R3, R4: value (none) -> 10k; footprint (none) -> Resistor_SMD:R_0201_0603Metric
- R5, R6: value (none) -> 1.2k 0.5%; footprint (none) -> Resistor_SMD:R_0201_0603Metric
- R7, R8: value (none) -> 100R; footprint (none) -> Resistor_SMD:R_0201_0603Metric
- TP1: value (none) -> BV0
- TP2: value (none) -> BV1
