File: module.kicad_sch (KiCad schematic)
At the start: 18 parts

Commit message: wip save
Parts:
- C38, C40: value (none) -> 1uF; footprint (none) -> Capacitor_SMD:C_0402_1005Metric
- C39, C41, C42, C43, C44, C45, C46, C47, C48, C? (x5): value (none) -> 0.1uF; footprint (none) -> Capacitor_SMD:C_0201_0603Metric
- R11: renamed from R10; value (none) -> 100R; footprint (none) -> Resistor_SMD:R_0201_0603Metric
- U4: renamed from U1; value (none) -> ETROCv2; footprint (none) -> etl_module_mockup:ETROCv2_64pad
